Commit message: Modified robot assets structure for X2 and created mjcf files.

File: resources/robots/x2/urdf/x2_ultra.urdf (robot description, URDF)
Before this commit: robot x2t2.5, 39 links, 38 joints
Links:
- added link base_link
- added link lidar_chest_front
- link head_pitch_link: geometry collision mesh filename=../meshes/head_pitch_link.STL; visual mesh filename=../meshes/head_pitch_link.STL
- link head_yaw_link: geometry collision mesh filename=../meshes/head_yaw_link.STL; visual mesh filename=../meshes/head_yaw_link.STL
- link imu_in_head_link: geometry visual mesh filename=../meshes/imu_in_head_link.STL
- link imu_in_pelvis_link: geometry visual mesh filename=../meshes/imu_in_pelvis_link.STL
- link imu_in_torso_link: geometry visual mesh filename=../meshes/imu_in_torso_link.STL
- link left_ankle_pitch_link: geometry collision mesh filename=../meshes/left_ankle_pitch_link.STL; visual mesh filename=../meshes/left_ankle_pitch_link.STL
- link left_ankle_roll_link: geometry collision mesh filename=../meshes/left_ankle_roll_link.STL; visual mesh filename=../meshes/left_ankle_roll_link.STL
- link left_elbow_link: geometry collision mesh filename=../meshes/left_elbow_link.STL; visual mesh filename=../meshes/left_elbow_link.STL
- link left_hip_pitch_link: geometry collision mesh filename=../meshes/left_hip_pitch_link.STL; visual mesh filename=../meshes/left_hip_pitch_link.STL
- link left_hip_roll_link: geometry collision mesh filename=../meshes/left_hip_roll_link.STL scale=1.0 0.9 1.0; visual mesh filename=../meshes/left_hip_roll_link.STL
- link left_hip_yaw_link: geometry collision mesh filename=../meshes/left_hip_yaw_link.STL; visual mesh filename=../meshes/left_hip_yaw_link.STL
- link left_knee_link: geometry collision mesh filename=../meshes/left_knee_link.STL; visual mesh filename=../meshes/left_knee_link.STL
- link left_shoulder_pitch_link: geometry collision mesh filename=../meshes/left_shoulder_pitch_link.STL; visual mesh filename=../meshes/left_shoulder_pitch_link.STL
- link left_shoulder_roll_link: geometry collision mesh filename=../meshes/left_shoulder_roll_link.STL; visual mesh filename=../meshes/left_shoulder_roll_link.STL
- link left_shoulder_yaw_link: geometry collision mesh filename=../meshes/left_shoulder_yaw_link.STL; visual mesh filename=../meshes/left_shoulder_yaw_link.STL
- link left_wrist_pitch_link: geometry collision mesh filename=../meshes/left_wrist_pitch_link.STL; visual mesh filename=../meshes/left_wrist_pitch_link.STL
- link left_wrist_roll_link: geometry collision mesh filename=../meshes/left_wrist_roll_link.STL; visual mesh filename=../meshes/left_wrist_roll_link.STL
- link left_wrist_yaw_link: geometry collision mesh filename=../meshes/left_wrist_yaw_link.STL; visual mesh filename=../meshes/left_wrist_yaw_link.STL
- link pelvis: geometry collision mesh filename=../meshes/pelvis.STL; visual mesh filename=../meshes/pelvis.STL
- link rgb_head_center: geometry visual mesh filename=../meshes/rgb_head_center_link.STL
- link rgb_head_rear: geometry visual mesh filename=../meshes/rgb_head_rear_link.STL
- link rgbd_head_front: geometry visual mesh filename=../meshes/rgbd_head_front_link.STL
- link right_ankle_pitch_link: geometry collision mesh filename=../meshes/right_ankle_pitch_link.STL; visual mesh filename=../meshes/right_ankle_pitch_link.STL
- link right_ankle_roll_link: geometry collision mesh filename=../meshes/right_ankle_roll_link.STL; visual mesh filename=../meshes/right_ankle_roll_link.STL
- link right_elbow_link: geometry collision mesh filename=../meshes/right_elbow_link.STL; visual mesh filename=../meshes/right_elbow_link.STL
- link right_hip_pitch_link: geometry collision mesh filename=../meshes/right_hip_pitch_link.STL; visual mesh filename=../meshes/right_hip_pitch_link.STL
- link right_hip_roll_link: geometry collision mesh filename=../meshes/right_hip_roll_link.STL scale=1.0 0.9 1.0; visual mesh filename=../meshes/right_hip_roll_link.STL
- link right_hip_yaw_link: geometry collision mesh filename=../meshes/right_hip_yaw_link.STL; visual mesh filename=../meshes/right_hip_yaw_link.STL
- link right_knee_link: geometry collision mesh filename=../meshes/right_knee_link.STL; visual mesh filename=../meshes/right_knee_link.STL
- link right_shoulder_pitch_link: geometry collision mesh filename=../meshes/right_shoulder_pitch_link.STL; visual mesh filename=../meshes/right_shoulder_pitch_link.STL
- link right_shoulder_roll_link: geometry collision mesh filename=../meshes/right_shoulder_roll_link.STL; visual mesh filename=../meshes/right_shoulder_roll_link.STL
- link right_shoulder_yaw_link: geometry collision mesh filename=../meshes/right_shoulder_yaw_link.STL; visual mesh filename=../meshes/right_shoulder_yaw_link.STL
- link right_wrist_pitch_link: geometry collision mesh filename=../meshes/right_wrist_pitch_link.STL; visual mesh filename=../meshes/right_wrist_pitch_link.STL
- link right_wrist_roll_link: geometry collision mesh filename=../meshes/right_wrist_roll_link.STL; visual mesh filename=../meshes/right_wrist_roll_link.STL
- link right_wrist_yaw_link: geometry collision mesh filename=../meshes/right_wrist_yaw_link.STL; visual mesh filename=../meshes/right_wrist_yaw_link.STL
- link stereo_head_front: geometry visual mesh filename=../meshes/stereo_head_front_link.STL
- link torso_link: geometry collision mesh filename=../meshes/torso_plus_link.STL; visual mesh filename=../meshes/torso_plus_link.STL
- link waist_pitch_link: geometry visual mesh filename=../meshes/waist_pitch_link.STL
- link waist_yaw_link: geometry visual mesh filename=../meshes/waist_yaw_link.STL
Joints:
- added joint base_link_joint: type fixed, parent base_link, child pelvis, origin xyz=0.0 0 0.0 rpy=0 0 0
- added joint lidar_chest_front: type fixed, parent torso_link, child lidar_chest_front, origin xyz=0.102632855873251 0 0.181586916322065 rpy=-1.5707963267949 0 0, axis 0 0 0
- joint head_pitch_joint: type fixed -> revolute
- joint head_yaw_joint: type fixed -> revolute
- joint left_elbow_joint: type fixed -> revolute
- joint left_shoulder_pitch_joint: type fixed -> revolute
- joint left_shoulder_roll_joint: type fixed -> revolute
- joint left_shoulder_yaw_joint: type fixed -> revolute
- joint left_wrist_pitch_joint: type fixed -> revolute
- joint left_wrist_roll_joint: type fixed -> revolute
- joint left_wrist_yaw_joint: type fixed -> revolute
- joint right_elbow_joint: type fixed -> revolute
- joint right_shoulder_pitch_joint: type fixed -> revolute
- joint right_shoulder_roll_joint: type fixed -> revolute
- joint right_shoulder_yaw_joint: type fixed -> revolute
- joint right_wrist_pitch_joint: type fixed -> revolute
- joint right_wrist_roll_joint: type fixed -> revolute
- joint right_wrist_yaw_joint: type fixed -> revolute

File: resources/robots/x2/urdf/x2_ultra_simple_collision.urdf (robot description, URDF)
Before this commit: robot x2t2.5, 41 links, 40 joints
Links:
- removed link base_link
- removed link lidar_chest_front
- link head_pitch_link: geometry visual mesh filename=../meshes/head_pitch_link.STL
- link head_yaw_link: geometry visual mesh filename=../meshes/head_yaw_link.STL
- link imu_in_head_link: geometry visual mesh filename=../meshes/imu_in_head_link.STL
- link imu_in_pelvis_link: geometry visual mesh filename=../meshes/imu_in_pelvis_link.STL
- link imu_in_torso_link: geometry visual mesh filename=../meshes/imu_in_torso_link.STL
- link left_ankle_pitch_link: geometry visual mesh filename=../meshes/left_ankle_pitch_link.STL
- link left_ankle_roll_link: geometry collision sphere radius=0.005; collision sphere radius=0.005
- link left_elbow_link: geometry collision cylinder length=0.09 radius=0.04; visual mesh filename=../meshes/left_elbow_link.STL
- link left_hip_pitch_link: geometry visual mesh filename=../meshes/left_hip_pitch_link.STL
- link left_hip_roll_link: geometry collision mesh filename=../meshes/left_hip_roll_link.STL scale=1.0 0.9 1.0; visual mesh filename=../meshes/left_hip_roll_link.STL
- link left_hip_yaw_link: geometry collision cylinder length=0.03 radius=0.042; collision cylinder length=0.03 radius=0.042
- link left_knee_link: geometry collision mesh filename=../meshes/left_knee_link.STL; visual mesh filename=../meshes/left_knee_link.STL
- link left_shoulder_pitch_link: geometry visual mesh filename=../meshes/left_shoulder_pitch_link.STL
- link left_shoulder_roll_link: geometry collision mesh filename=../meshes/left_shoulder_roll_link.STL; visual mesh filename=../meshes/left_shoulder_roll_link.STL
- link left_shoulder_yaw_link: geometry collision cylinder length=0.024 radius=0.028; collision cylinder length=0.05 radius=0.042
- link left_wrist_pitch_link: geometry visual mesh filename=../meshes/left_wrist_pitch_link.STL
- link left_wrist_roll_link: geometry collision box size=0.07 0.045 0.14; visual mesh filename=../meshes/left_wrist_roll_link.STL
- link left_wrist_yaw_link: geometry collision mesh filename=../meshes/left_wrist_yaw_link.STL; visual mesh filename=../meshes/left_wrist_yaw_link.STL
- link pelvis: geometry collision mesh filename=../meshes/pelvis.STL; visual mesh filename=../meshes/pelvis.STL
- link rgb_head_center: geometry visual mesh filename=../meshes/rgb_head_center_link.STL
- link rgb_head_rear: geometry visual mesh filename=../meshes/rgb_head_rear_link.STL
- link rgbd_head_front: geometry visual mesh filename=../meshes/rgbd_head_front_link.STL
- link right_ankle_pitch_link: geometry visual mesh filename=../meshes/right_ankle_pitch_link.STL
- link right_ankle_roll_link: geometry collision sphere radius=0.005; collision sphere radius=0.005
- link right_elbow_link: geometry collision cylinder length=0.09 radius=0.04; visual mesh filename=../meshes/right_elbow_link.STL
- link right_hip_pitch_link: geometry visual mesh filename=../meshes/right_hip_pitch_link.STL
- link right_hip_roll_link: geometry collision mesh filename=../meshes/right_hip_roll_link.STL scale=1.0 0.9 1.0; visual mesh filename=../meshes/right_hip_roll_link.STL
- link right_hip_yaw_link: geometry collision cylinder length=0.03 radius=0.042; collision cylinder length=0.03 radius=0.042
- link right_knee_link: geometry collision mesh filename=../meshes/right_knee_link.STL; visual mesh filename=../meshes/right_knee_link.STL
- link right_shoulder_pitch_link: geometry visual mesh filename=../meshes/right_shoulder_pitch_link.STL
- link right_shoulder_roll_link: geometry collision mesh filename=../meshes/right_shoulder_roll_link.STL; visual mesh filename=../meshes/right_shoulder_roll_link.STL
- link right_shoulder_yaw_link: geometry collision cylinder length=0.024 radius=0.028; collision cylinder length=0.05 radius=0.042
- link right_wrist_pitch_link: geometry visual mesh filename=../meshes/right_wrist_pitch_link.STL
- link right_wrist_roll_link: geometry collision box size=0.07 0.045 0.14; visual mesh filename=../meshes/right_wrist_roll_link.STL
- link right_wrist_yaw_link: geometry collision mesh filename=../meshes/right_wrist_yaw_link.STL; visual mesh filename=../meshes/right_wrist_yaw_link.STL
- link stereo_head_front: geometry visual mesh filename=../meshes/stereo_head_front_link.STL
- link torso_link: geometry collision mesh filename=../meshes/torso_plus_link.STL; visual mesh filename=../meshes/torso_plus_link.STL
- link waist_pitch_link: geometry visual mesh filename=../meshes/waist_pitch_link.STL
- link waist_yaw_link: geometry visual mesh filename=../meshes/waist_yaw_link.STL
Joints:
- removed joint base_link_joint
- removed joint lidar_chest_front
