Commit message: The x2 urdf and mjcf files have been modified to only control lower body joints.

File: resources/robots/x2/urdf/x2_ultra_simple_collision.urdf (robot description, URDF)
Before this commit: robot x2t2.5, 39 links, 38 joints
Joints:
- joint head_pitch_joint: type revolute -> fixed
- joint head_yaw_joint: type revolute -> fixed
- joint left_elbow_joint: type revolute -> fixed
- joint left_shoulder_pitch_joint: type revolute -> fixed
- joint left_shoulder_roll_joint: type revolute -> fixed
- joint left_shoulder_yaw_joint: type revolute -> fixed
- joint left_wrist_pitch_joint: type revolute -> fixed
- joint left_wrist_roll_joint: type revolute -> fixed
- joint left_wrist_yaw_joint: type revolute -> fixed
- joint right_elbow_joint: type revolute -> fixed
- joint right_shoulder_pitch_joint: type revolute -> fixed
- joint right_shoulder_roll_joint: type revolute -> fixed
- joint right_shoulder_yaw_joint: type revolute -> fixed
- joint right_wrist_pitch_joint: type revolute -> fixed
- joint right_wrist_roll_joint: type revolute -> fixed
- joint right_wrist_yaw_joint: type revolute -> fixed
- joint waist_pitch_joint: type revolute -> fixed
- joint waist_roll_joint: type revolute -> fixed
- joint waist_yaw_joint: type revolute -> fixed
